Commit message: Reshape the arm as an IRB-1200-class machine and model its six drives
The model was a stack of plain cylinders with placeholder dimensions. It is
now a proper industrial arm, built entirely from primitives - no vendor
mesh, badge or branding, and no affiliation with ABB.

Geometry
  * kinematics: 0.899 m reach, axis 2 at 0.399 m, 0.082 m wrist-to-flange,
    all derived from one `kinematics:` block so the chain can never drift
    from the geometry that is drawn
  * a cranked elbow - the forearm is offset 42 mm from the elbow axis,
    which is the signature a coaxial model gets wrong
  * composite links: cast base, rotating column with a shoulder shaft,
    tapered upper arm, tubular forearm, compact three-roll wrist, 63 mm
    tool flange
  * the spherical wrist is preserved and now asserted by a test: axes 4/5/6
    intersect at the joint_5 origin
  * industrial palette - orange castings, graphite housings, black drives

Drive units
  * six servo + gearbox assemblies as real links with mass and inertia,
    mounted on the links that carry them, from a `motors:` block
  * 11.5 kg of the arm's 51.9 kg, most of it high on the moving links;
    leaving it out makes a simulated arm accelerate in ways the real one
    cannot
  * no collision geometry by default: they sit inside the arm's own
    envelope, so checking them costs planning time and changes no result
  * their motor_id is the id the driver addresses on the bus, and a test
    fails the build if the model and the driver ever disagree
  * use_motors:=false gives a lighter, purely kinematic arm

Envelope, limits and drive train, all consistent by test
  * joint ranges and speeds of the intended machine (axis 1 +-170 deg at
    288 deg/s through axis 6 +-400 deg at 600 deg/s)
  * MoveIt limits, the safety monitor and the calibration file regenerated
    from robot.yaml, so none of them can exceed the mechanical limits
  * gear ratios, encoder resolutions (17-bit main axes, 16-bit wrist),
    torque constants and current limits sized so every joint's rated
    effort is actually deliverable - a new test proves it, and another
    checks the wrist is faster and more lightly geared than the main axes

Tooling
  * scripts/urdf_preview.py renders the model to a PNG with no RViz, no
    Gazebo and no display, by doing its own forward kinematics.  It is how
    this geometry was debugged: it caught the base drive intersecting the
    rotating column's sweep, which was then remounted on the column

85 python tests (was 72) and the 53 C++ cases pass; the model expands in
all three backends, with and without drives, and with a frame prefix.

Co-Authored-By: Claude Opus 5 <noreply@anthropic.com>
Claude-Session: https://claude.ai/code/session_01UhhpSXFHQi2psSUYcgzj2W

File: robot_arm_ws/src/robot_arm_description/urdf/gazebo.xacro (robot description, xacro)
@@ -31,21 +31,37 @@
   </xacro:macro>
   <xacro:macro name="robot_arm_gazebo"
-               params="prefix sim_engine robot_config_file controllers_file">
+               params="prefix sim_engine robot_config_file controllers_file use_motors:=true">
     <xacro:property name="cfg" value="${xacro.load_yaml(robot_config_file)}"/>
     <xacro:property name="gz" value="${cfg['gazebo']}"/>
     <xacro:arm_gazebo_link name="${prefix}base_link" material="${gz['base_material']}"
       mu1="${gz['mu1']}" mu2="${gz['mu2']}" self_collide="${gz['self_collide']}"/>
-    <xacro:arm_gazebo_link name="${prefix}link_1" material="${gz['joint_material']}"
+    <xacro:arm_gazebo_link name="${prefix}link_1" material="${gz['link_material']}"
       mu1="${gz['mu1']}" mu2="${gz['mu2']}" self_collide="${gz['self_collide']}"/>
     <xacro:arm_gazebo_link name="${prefix}link_2" material="${gz['link_material']}"
       mu1="${gz['mu1']}" mu2="${gz['mu2']}" self_collide="${gz['self_collide']}"/>
-    <xacro:arm_gazebo_link name="${prefix}link_3" material="${gz['joint_material']}"
+    <xacro:arm_gazebo_link name="${prefix}link_3" material="${gz['link_material']}"
       mu1="${gz['mu1']}" mu2="${gz['mu2']}" self_collide="${gz['self_collide']}"/>
-    <xacro:arm_gazebo_link name="${prefix}link_4" material="${gz['link_material']}"
+    <xacro:arm_gazebo_link name="${prefix}link_4" material="${gz['wrist_material']}"
       mu1="${gz['mu1']}" mu2="${gz['mu2']}" self_collide="${gz['self_collide']}"/>
-    <xacro:arm_gazebo_link name="${prefix}link_5" material="${gz['joint_material']}"
+    <xacro:arm_gazebo_link name="${prefix}link_5" material="${gz['wrist_material']}"
       mu1="${gz['mu1']}" mu2="${gz['mu2']}" self_collide="${gz['self_collide']}"/>
-    <xacro:arm_gazebo_link name="${prefix}link_6" material="${gz['base_material']}"
+    <xacro:arm_gazebo_link name="${prefix}link_6" material="${gz['joint_material']}"
       mu1="${gz['mu1']}" mu2="${gz['mu2']}" self_collide="${gz['self_collide']}"/>
+    <!-- Drive units.  They carry mass in the physics engine either way; this
+         only decides how they are shaded. -->
+    <xacro:if value="${use_motors}">
+      <xacro:arm_gazebo_link name="${prefix}motor_1" material="${gz['motor_material']}"
+        mu1="${gz['mu1']}" mu2="${gz['mu2']}" self_collide="false"/>
+      <xacro:arm_gazebo_link name="${prefix}motor_2" material="${gz['motor_material']}"
+        mu1="${gz['mu1']}" mu2="${gz['mu2']}" self_collide="false"/>
+      <xacro:arm_gazebo_link name="${prefix}motor_3" material="${gz['motor_material']}"
+        mu1="${gz['mu1']}" mu2="${gz['mu2']}" self_collide="false"/>
+      <xacro:arm_gazebo_link name="${prefix}motor_4" material="${gz['motor_material']}"
+        mu1="${gz['mu1']}" mu2="${gz['mu2']}" self_collide="false"/>
+      <xacro:arm_gazebo_link name="${prefix}motor_5" material="${gz['motor_material']}"
+        mu1="${gz['mu1']}" mu2="${gz['mu2']}" self_collide="false"/>
+      <xacro:arm_gazebo_link name="${prefix}motor_6" material="${gz['motor_material']}"
+        mu1="${gz['mu1']}" mu2="${gz['mu2']}" self_collide="false"/>
+    </xacro:if>
     <xacro:arm_gazebo_joint name="${prefix}joint_1"/>
     <xacro:arm_gazebo_joint name="${prefix}joint_2"/>

File: robot_arm_ws/src/robot_arm_description/urdf/inertials.xacro (robot description, xacro)
@@ -34,3 +34,22 @@
     </inertial>
   </xacro:macro>
+  <!-- Build a link's inertial from its `inertial:` entry in robot.yaml.
+       A URDF link carries exactly one inertial, so a composite link declares
+       the equivalent solid its tensor is derived from and where its centre of
+       mass sits. -->
+  <xacro:macro name="link_inertial" params="spec">
+    <xacro:if value="${spec['shape'] == 'cylinder'}">
+      <xacro:cylinder_inertial
+        mass="${spec['mass']}" radius="${spec['radius']}" length="${spec['length']}">
+        <origin xyz="${spec['com'][0]} ${spec['com'][1]} ${spec['com'][2]}" rpy="0 0 0"/>
+      </xacro:cylinder_inertial>
+    </xacro:if>
+    <xacro:if value="${spec['shape'] == 'box'}">
+      <xacro:box_inertial
+        mass="${spec['mass']}"
+        x="${spec['size'][0]}" y="${spec['size'][1]}" z="${spec['size'][2]}">
+        <origin xyz="${spec['com'][0]} ${spec['com'][1]} ${spec['com'][2]}" rpy="0 0 0"/>
+      </xacro:box_inertial>
+    </xacro:if>
+  </xacro:macro>
 </robot>

File: robot_arm_ws/src/robot_arm_description/urdf/materials.xacro (robot description, xacro)
@@ -1,20 +1,36 @@
 <?xml version="1.0"?>
 <!--
-  RViz / URDF materials.  Gazebo materials are applied separately in
-  gazebo.xacro because Gazebo Classic ignores <material> tags coming from URDF.
+  RViz / URDF materials.
+  The palette is the industrial-arm convention: an orange arm on a graphite
+  base and wrist, with black drive units.  Gazebo materials are applied
+  separately in gazebo.xacro, because Gazebo Classic ignores <material> tags
+  that come from URDF.
 -->
 <robot xmlns:xacro="http://www.ros.org/wiki/xacro">
-  <material name="arm_dark_grey">
-    <color rgba="0.25 0.25 0.27 1.0"/>
+  <!-- Arm castings. -->
+  <material name="arm_orange">
+    <color rgba="1.00 0.42 0.07 1.0"/>
   </material>
-  <material name="arm_grey">
-    <color rgba="0.72 0.72 0.74 1.0"/>
+  <!-- Base, joint housings and yokes. -->
+  <material name="arm_graphite">
+    <color rgba="0.24 0.25 0.27 1.0"/>
   </material>
-  <material name="arm_orange">
-    <color rgba="0.95 0.55 0.10 1.0"/>
+  <!-- Wrist castings. -->
+  <material name="arm_light_grey">
+    <color rgba="0.72 0.73 0.75 1.0"/>
   </material>
-  <material name="arm_black">
-    <color rgba="0.08 0.08 0.08 1.0"/>
+  <!-- Machined tool flange. -->
+  <material name="arm_steel">
+    <color rgba="0.55 0.56 0.58 1.0"/>
   </material>
+  <!-- Motor bodies. -->
+  <material name="motor_black">
+    <color rgba="0.10 0.10 0.11 1.0"/>
+  </material>
+  <!-- Gearbox housings. -->
+  <material name="gearbox_grey">
+    <color rgba="0.38 0.39 0.41 1.0"/>
+  </material>
+  <!-- Gripper mounting plate. -->
   <material name="arm_blue">
     <color rgba="0.15 0.35 0.75 1.0"/>

File: robot_arm_ws/src/robot_arm_description/urdf/robot_arm.urdf.xacro (robot description, xacro)
@@ -36,4 +36,7 @@
   <!-- Optional gripper mounting plate + tool_tip frame. -->
   <xacro:arg name="use_gripper_mount" default="true"/>
+  <!-- Model the six servo/gearbox drive units as links with mass.  Turning
+       them off gives a lighter, purely kinematic arm. -->
+  <xacro:arg name="use_motors" default="true"/>
   <!-- Emit <transmission> entries (see transmissions.xacro). -->
   <xacro:arg name="use_transmissions" default="false"/>
@@ -71,5 +74,6 @@
     prefix="${prefix}"
     robot_config_file="$(arg robot_config_file)"
-    use_gripper_mount="$(arg use_gripper_mount)"/>
+    use_gripper_mount="$(arg use_gripper_mount)"
+    use_motors="$(arg use_motors)"/>
   <!-- ===================== ros2_control =============================== -->
   <xacro:robot_arm_ros2_control
@@ -89,5 +93,6 @@
       sim_engine="${sim_engine}"
       robot_config_file="$(arg robot_config_file)"
-      controllers_file="$(arg controllers_file)"/>
+      controllers_file="$(arg controllers_file)"
+      use_motors="$(arg use_motors)"/>
   </xacro:if>
 </robot>
