Commit message: Compute real inertia tensors from the geometry instead of faking them
A URDF link carries one inertial, which makes a composite link easy to fake
with a single equivalent solid - and that is what this model did.  link_3 is
a forearm tube offset 42 mm in X plus a shaft lying across Y, but it was
given a centred cylinder: every product of inertia zero, and a centre of mass
guessed by hand.  A physics engine integrates those numbers, so the simulated
arm swung about axes the real one does not and fought torques the machine
never produces.

scripts/compute_inertia.py treats each link's visual primitives as one rigid
body of uniform density, derives that density from the link's target mass in
robot.yaml, and sums the parts with the parallel axis theorem: centre of mass,
principal moments and products of inertia.  The result is generated into
config/inertia.yaml, which the model now loads; masses stay a design input.

For link_3 the correction is not cosmetic:

    centre of mass z   0.170  ->  0.115   (48% error in the moment arm)
    ixx                0.0750 ->  0.1028
    izz                0.0099 ->  0.0155
    ixz                0.0    -> -0.0110  (a coupling that did not exist)

Four tests.  Every tensor is checked positive definite and against the
triangle inequality on its principal moments - a body violating either cannot
exist, and engines answer with instability rather than an error; all 14 pass.
link_3 must carry a product of inertia, so nobody can quietly reinstate an
equivalent solid.  Centres of mass must lie inside their geometry.  And the
generator is re-run and diffed against the committed file, so changing a
dimension without regenerating fails the build instead of leaving the model
with the inertia of a robot that no longer exists.

Co-Authored-By: Claude Opus 5 <noreply@anthropic.com>
Claude-Session: https://claude.ai/code/session_01UhhpSXFHQi2psSUYcgzj2W

File: robot_arm_ws/src/robot_arm_description/urdf/inertials.xacro (robot description, xacro)
@@ -1,55 +1,30 @@
 <?xml version="1.0"?>
 <!--
-  Reusable inertial macros.  Using analytic inertia tensors of primitive solids
-  keeps the model physically plausible without a CAD export, and keeps Gazebo
-  numerically stable (no zero or negative principal moments).
+  Inertial properties.
+  A URDF link carries exactly one inertial, which makes it easy to fake a
+  composite link with a single equivalent solid.  This model does not: the
+  tensors come from config/inertia.yaml, where scripts/compute_inertia.py
+  writes them after summing each link's actual primitives with the parallel
+  axis theorem - centre of mass, principal moments and products of inertia.
+  Regenerate after any change to geometry or mass:
+    xacro urdf/robot_arm.urdf.xacro > /tmp/arm.urdf
+    ros2 run robot_arm_description compute_inertia.py /tmp/arm.urdf \
+        config/robot.yaml > config/inertia.yaml
+  A test regenerates the file and fails if it no longer matches the geometry,
+  so the two cannot drift apart silently.
 -->
 <robot xmlns:xacro="http://www.ros.org/wiki/xacro">
-  <!-- Solid cylinder extruded along its own +Z axis. -->
-  <xacro:macro name="cylinder_inertial" params="mass radius length *origin">
+  <xacro:macro name="link_inertial" params="spec">
     <inertial>
-      <xacro:insert_block name="origin"/>
-      <mass value="${mass}"/>
+      <origin xyz="${spec['com'][0]} ${spec['com'][1]} ${spec['com'][2]}" rpy="0 0 0"/>
+      <mass value="${spec['mass']}"/>
       <inertia
-        ixx="${(mass * (3.0 * radius * radius + length * length)) / 12.0}"
-        ixy="0.0"
-        ixz="0.0"
-        iyy="${(mass * (3.0 * radius * radius + length * length)) / 12.0}"
-        iyz="0.0"
-        izz="${(mass * radius * radius) / 2.0}"/>
+        ixx="${spec['inertia']['ixx']}"
+        ixy="${spec['inertia']['ixy']}"
+        ixz="${spec['inertia']['ixz']}"
+        iyy="${spec['inertia']['iyy']}"
+        iyz="${spec['inertia']['iyz']}"
+        izz="${spec['inertia']['izz']}"/>
     </inertial>
   </xacro:macro>
-  <!-- Solid box. -->
-  <xacro:macro name="box_inertial" params="mass x y z *origin">
-    <inertial>
-      <xacro:insert_block name="origin"/>
-      <mass value="${mass}"/>
-      <inertia
-        ixx="${(mass * (y * y + z * z)) / 12.0}"
-        ixy="0.0"
-        ixz="0.0"
-        iyy="${(mass * (x * x + z * z)) / 12.0}"
-        iyz="0.0"
-        izz="${(mass * (x * x + y * y)) / 12.0}"/>
-    </inertial>
-  </xacro:macro>
-  <!-- Build a link's inertial from its `inertial:` entry in robot.yaml.
-       A URDF link carries exactly one inertial, so a composite link declares
-       the equivalent solid its tensor is derived from and where its centre of
-       mass sits. -->
-  <xacro:macro name="link_inertial" params="spec">
-    <xacro:if value="${spec['shape'] == 'cylinder'}">
-      <xacro:cylinder_inertial
-        mass="${spec['mass']}" radius="${spec['radius']}" length="${spec['length']}">
-        <origin xyz="${spec['com'][0]} ${spec['com'][1]} ${spec['com'][2]}" rpy="0 0 0"/>
-      </xacro:cylinder_inertial>
-    </xacro:if>
-    <xacro:if value="${spec['shape'] == 'box'}">
-      <xacro:box_inertial
-        mass="${spec['mass']}"
-        x="${spec['size'][0]}" y="${spec['size'][1]}" z="${spec['size'][2]}">
-        <origin xyz="${spec['com'][0]} ${spec['com'][1]} ${spec['com'][2]}" rpy="0 0 0"/>
-      </xacro:box_inertial>
-    </xacro:if>
-  </xacro:macro>
 </robot>

File: robot_arm_ws/src/robot_arm_description/urdf/motors.xacro (robot description, xacro)
@@ -21,5 +21,5 @@
 -->
 <robot xmlns:xacro="http://www.ros.org/wiki/xacro">
-  <xacro:macro name="drive_unit" params="name parent spec use_collision">
+  <xacro:macro name="drive_unit" params="name parent spec inertial use_collision">
     <link name="${name}">
       <!-- Gearbox: the wide, short housing bolted to the link. -->
@@ -48,11 +48,7 @@
         </collision>
       </xacro:if>
-      <!-- One inertial for the whole assembly, about its combined centre. -->
-      <xacro:cylinder_inertial
-        mass="${spec['mass']}"
-        radius="${spec['gearbox_radius']}"
-        length="${spec['gearbox_length'] + spec['length']}">
-        <origin xyz="0 0 ${(spec['gearbox_length'] + spec['length']) / 2.0}" rpy="0 0 0"/>
-      </xacro:cylinder_inertial>
+      <!-- Gearbox and motor body summed into one tensor about their combined
+           centre of mass; see inertials.xacro. -->
+      <xacro:link_inertial spec="${inertial}"/>
     </link>
     <joint name="${name}_mount" type="fixed">
@@ -65,17 +61,23 @@
   </xacro:macro>
   <!-- All six drives, mounted on the links named in robot.yaml. -->
-  <xacro:macro name="robot_arm_motors" params="prefix motors">
+  <xacro:macro name="robot_arm_motors" params="prefix motors inertia">
     <xacro:drive_unit name="${prefix}motor_1" parent="${prefix}${motors['joint_1']['parent']}"
-                      spec="${motors['joint_1']}" use_collision="${motors['use_collision']}"/>
+                      spec="${motors['joint_1']}" inertial="${inertia['motor_1']}"
+                      use_collision="${motors['use_collision']}"/>
     <xacro:drive_unit name="${prefix}motor_2" parent="${prefix}${motors['joint_2']['parent']}"
-                      spec="${motors['joint_2']}" use_collision="${motors['use_collision']}"/>
+                      spec="${motors['joint_2']}" inertial="${inertia['motor_2']}"
+                      use_collision="${motors['use_collision']}"/>
     <xacro:drive_unit name="${prefix}motor_3" parent="${prefix}${motors['joint_3']['parent']}"
-                      spec="${motors['joint_3']}" use_collision="${motors['use_collision']}"/>
+                      spec="${motors['joint_3']}" inertial="${inertia['motor_3']}"
+                      use_collision="${motors['use_collision']}"/>
     <xacro:drive_unit name="${prefix}motor_4" parent="${prefix}${motors['joint_4']['parent']}"
-                      spec="${motors['joint_4']}" use_collision="${motors['use_collision']}"/>
+                      spec="${motors['joint_4']}" inertial="${inertia['motor_4']}"
+                      use_collision="${motors['use_collision']}"/>
     <xacro:drive_unit name="${prefix}motor_5" parent="${prefix}${motors['joint_5']['parent']}"
-                      spec="${motors['joint_5']}" use_collision="${motors['use_collision']}"/>
+                      spec="${motors['joint_5']}" inertial="${inertia['motor_5']}"
+                      use_collision="${motors['use_collision']}"/>
     <xacro:drive_unit name="${prefix}motor_6" parent="${prefix}${motors['joint_6']['parent']}"
-                      spec="${motors['joint_6']}" use_collision="${motors['use_collision']}"/>
+                      spec="${motors['joint_6']}" inertial="${inertia['motor_6']}"
+                      use_collision="${motors['use_collision']}"/>
   </xacro:macro>
 </robot>

File: robot_arm_ws/src/robot_arm_description/urdf/robot_arm.urdf.xacro (robot description, xacro)
@@ -45,4 +45,6 @@
   <xacro:arg name="robot_config_file"
              default="$(find robot_arm_description)/config/robot.yaml"/>
+  <xacro:arg name="inertia_file"
+             default="$(find robot_arm_description)/config/inertia.yaml"/>
   <xacro:arg name="initial_positions_file"
              default="$(find robot_arm_description)/config/initial_positions.yaml"/>
@@ -74,4 +76,5 @@
     prefix="${prefix}"
     robot_config_file="$(arg robot_config_file)"
+    inertia_file="$(arg inertia_file)"
     use_gripper_mount="$(arg use_gripper_mount)"
     use_motors="$(arg use_motors)"/>

File: robot_arm_ws/src/robot_arm_description/urdf/robot_arm_macro.xacro (robot description, xacro)
@@ -86,10 +86,11 @@
        The arm itself.
        ===================================================================== -->
-  <xacro:macro name="robot_arm" params="prefix robot_config_file use_gripper_mount:=true
-                                        use_motors:=true">
+  <xacro:macro name="robot_arm" params="prefix robot_config_file inertia_file
+                                        use_gripper_mount:=true use_motors:=true">
     <xacro:property name="cfg" value="${xacro.load_yaml(robot_config_file)}"/>
+    <!-- Tensors computed from the real geometry; see inertials.xacro. -->
+    <xacro:property name="inr" value="${xacro.load_yaml(inertia_file)['inertial']}"/>
     <xacro:property name="kin" value="${cfg['kinematics']}"/>
     <xacro:property name="geom" value="${cfg['geometry']}"/>
-    <xacro:property name="inr" value="${cfg['inertial']}"/>
     <xacro:property name="jnt" value="${cfg['joints']}"/>
     <xacro:property name="grip" value="${cfg['gripper_mount']}"/>
@@ -256,5 +257,5 @@
     <!-- ================================================================ -->
     <xacro:if value="${use_motors}">
-      <xacro:robot_arm_motors prefix="${prefix}" motors="${cfg['motors']}"/>
+      <xacro:robot_arm_motors prefix="${prefix}" motors="${cfg['motors']}" inertia="${inr}"/>
     </xacro:if>
     <!-- ================================================================ -->
@@ -268,10 +269,5 @@
           xyz="0 0 ${grip['plate_thickness'] / 2.0}"
           material="arm_blue"/>
-        <xacro:cylinder_inertial
-          mass="${grip['plate_mass']}"
-          radius="${grip['plate_radius']}"
-          length="${grip['plate_thickness']}">
-          <origin xyz="0 0 ${grip['plate_thickness'] / 2.0}" rpy="0 0 0"/>
-        </xacro:cylinder_inertial>
+        <xacro:link_inertial spec="${inr['gripper_mount_link']}"/>
       </link>
       <joint name="${prefix}joint_gripper_mount" type="fixed">
